File: KiCad/ModeltrainWagonLight2/Modelwagonlight.sch (KiCad schematic (older format))
At the start: 16 parts, among them J1 Conn_01x01, J2 Conn_01x01, J3 Conn_01x01, J4 Conn_01x01, U1 LP2951DR

Commit message: Added TrackModbusMaster2.X with PIC18F25K40 (later 70). Set Modbus communication speed to 1Mbps. Therfore also the Trackmodbusmaster needs to be updated. To do: - get Trackmodbusmaster2 to work - Check if possible to hold slaves on receive interrupt to wait until a full message is received - check with the 18F series how the interrupt response looks like and try to get comm speed up and message / sec
Parts:
- C1: value 22u -> 10u
- C2: value 22u -> 4.7u
Changed lines of the file:
@@
 P 5600 4300
 F 0 "C1" H 5625 4400 50  0000 L CNN
-F 1 "22u" H 5625 4200 50  0000 L CNN
+F 1 "10u" H 5625 4200 50  0000 L CNN
 F 2 "Capacitor_SMD:C_1206_3216Metric" H 5638 4150 50  0001 C CNN
 F 3 "http://www.farnell.com/datasheets/2079197.pdf?_ga=2.237228869.453305454.1544563035-1187106011.1538513614&_gac=1.262713726.1544645790.Cj0KCQiAgMPgBRDDARIsAOh3uyJWgmg4Jmz9qsKK7EVWh3ooL0QXFRR6pElfBGS6pZkWxoBnou2jGrYaAp9cEALw_wcB" H 5600 4300 50  0001 C CNN
@@
 P 8700 4250
 F 0 "C2" H 8725 4350 50  0000 L CNN
-F 1 "22u" H 8725 4150 50  0000 L CNN
+F 1 "4.7u" H 8725 4150 50  0000 L CNN
 F 2 "Capacitor_SMD:C_1206_3216Metric" H 8738 4100 50  0001 C CNN
 F 3 "http://www.farnell.com/datasheets/2079197.pdf?_ga=2.237228869.453305454.1544563035-1187106011.1538513614&_gac=1.262713726.1544645790.Cj0KCQiAgMPgBRDDARIsAOh3uyJWgmg4Jmz9qsKK7EVWh3ooL0QXFRR6pElfBGS6pZkWxoBnou2jGrYaAp9cEALw_wcB" H 8700 4250 50  0001 C CNN
