File: KiCad/TrackAmplifier2/TrackAmplifier.sch (KiCad schematic (older format))
At the start: 119 parts, among them J1 DB15_Male_MountingHoles, J2 Conn_01x06, Q1 NTR5103NT1G, U1 ST485EBDR, U10 MCP1525, U11 MCP9701A-E/TO, U2 ST485EBDR, U3 L78M05CDT-1-TO-251-3, U4 LMD18200, U5 ST485EBDR, U6 ST485EBDR, U7 MCP6N11, U8 INA2180, U9 PIC18F25K40

Commit message: Updated SMD elco in order nr and manufacturer nr to fit on the board.
Parts:
- C21: Farnell (none) -> 2611386; Manufacturer nr MCGPR35V477M10X21 -> MCVVT035M221FB3L
Changed lines of the file:
@@
 F 1 "220u" H 1650 1150 50  0000 L CNN
 F 2 "Capacitor_SMD:CP_Elec_8x10.5" H 1988 900 50  0001 C CNN
-F 3 "" H 1950 1050 50  0001 C CNN
-F 4 "MCGPR35V477M10X21" H 1950 1050 50  0001 C CNN "Manufacturer nr"
+F 3 "http://www.farnell.com/datasheets/2151198.pdf?_ga=2.35239009.157561629.1548106566-1187106011.1538513614&_gac=1.190289369.1545668388.Cj0KCQiApILhBRD1ARIsAOXWTztLrOL1UeBtZiE8BOA0caa3FLfEzalbJeV0DPq3mYz4wfvUG7ZLprQaApwnEALw_wcB" H 1950 1050 50  0001 C CNN
+F 4 "MCVVT035M221FB3L" H 1950 1050 50  0001 C CNN "Manufacturer nr"
+F 5 "2611386" H 1950 1050 50  0001 C CNN "Farnell"
 	1    1950 1050
 	1    0    0    -1
