File: KiCad/PIC32MZ_piggyback/PIC32MZ_piggyback1/PIC32MZ_piggyback.sch (KiCad schematic (older format))
At the start: 12 parts, among them J1 Conn_02x13_Odd_Even, J1-1 Conn_01x13_Male, J1-2 Conn_01x13_Male, J2 Conn_02x13_Odd_Even, J2-1 Conn_01x13_Male, J2-2 Conn_01x13_Male, J3 Conn_02x13_Odd_Even, J3-1 Conn_01x13_Male, J3-2 Conn_01x13_Male, J4 Conn_02x13_Odd_Even, J4-1 Conn_01x13_Male, J4-2 Conn_01x13_Male

Commit message: Fault in PB1 --> renamed, and continued with the first version.
Connections:
- net labels added: MCLR, RB6, RB7, RXN, RXP, TXN, TXP, VCC
Other:
- note added: "Jx-1 = outside dubbel row connector\nJx-2 = inside dubbel row connector"
Changed lines of the file:
@@
 U 1 1 5C9B0ADF
 P 4850 3700
-F 0 "J1" H 4900 4517 50  0000 C CNN
-F 1 "Conn_02x13_Odd_Even" H 4900 4426 50  0000 C CNN
+F 0 "J1" H 4900 4600 50  0000 C CNN
+F 1 "Conn_02x13_Odd_Even" H 4750 4550 50  0000 C CNN
 F 2 "Connector_PinHeader_2.54mm:PinHeader_2x13_P2.54mm_Vertical" H 4850 3700 50  0001 C CNN
 F 3 "~" H 4850 3700 50  0001 C CNN
@@
 U 1 1 5C9B0AE6
 P 5650 3700
-F 0 "J1-2" H 5756 4478 50  0000 C CNN
-F 1 "Conn_01x13_Male" H 5756 4387 50  0000 C CNN
+F 0 "J1-2" H 5750 4600 50  0000 C CNN
+F 1 "Conn_01x13_Male" H 5750 4550 50  0000 C CNN
 F 2 "Connector_PinHeader_2.54mm:PinHeader_1x13_P2.54mm_Vertical" H 5650 3700 50  0001 C CNN
 F 3 "~" H 5650 3700 50  0001 C CNN
@@
 Text Label 2700 1650 0    50   ~ 0
 GND
+Text Notes 3100 2750 0    50   ~ 0
+Jx-1 = outside dubbel row connector\nJx-2 = inside dubbel row connector
+Text Label 1750 3700 0    50   ~ 0
+MCLR
+Text Label 1750 3900 0    50   ~ 0
+VCC
+Text Label 5250 1350 0    50   ~ 0
+VCC
+Text Label 5250 1750 0    50   ~ 0
+VCC
+Text Label 4300 1450 0    50   ~ 0
+VCC
+Text Label 1750 2450 0    50   ~ 0
+VCC
+Text Label 1750 1650 0    50   ~ 0
+VCC
+Text Label 2700 1750 0    50   ~ 0
+VCC
+Text Label 4350 3600 0    50   ~ 0
+VCC
+Text Label 4350 3100 0    50   ~ 0
+VCC
+Text Label 5250 3300 0    50   ~ 0
+VCC
+Text Label 5250 3100 0    50   ~ 0
+TXN
+Text Label 2700 2350 0    50   ~ 0
+RXP
+Text Label 1750 2350 0    50   ~ 0
+RXN
+Text Label 4350 3200 0    50   ~ 0
+TXP
+Text Label 1750 2050 0    50   ~ 0
+RB6
+Text Label 1750 1550 0    50   ~ 0
+RB7
 $EndSCHEMATC

Commit message: updated new piggyback1 pcb.
Connections:
- net labels added: LED1, LED2, MCU_MISO, MCU_MOSI, MCU_SCK, RA0, RA1, RA10, RA14, RA15, RA2, RA3, RA4, RA5, RA9, RB0, RB1, RB10, RB11, RB12, RB13, RB14, RB15, RB2, RB3, RB4, RB5, RB8, RB9, RC1, RC2, RC3, RC4, RD0, RD1, RD10, RD12, RD13, RD14, RD2, RD3, RD4, RD5, RD7, RD9, RE0, RE2, RE3, RE7, RE8, RE9, RF0, RF1, RF12, RF3, RF4, RF5, RG12, RG14, RG6, RG7, RG8, RG9
Changed lines of the file:
@@
 Text Label 1750 1550 0    50   ~ 0
 RB7
+Text Label 1750 3200 0    50   ~ 0
+LED1
+Text Label 1750 3300 0    50   ~ 0
+LED2
+Text Label 1750 3400 0    50   ~ 0
+RA9
+Text Label 1750 3500 0    50   ~ 0
+RB8
+Text Label 1750 3600 0    50   ~ 0
+RB10
+Text Label 1750 4000 0    50   ~ 0
+RB12
+Text Label 1750 4100 0    50   ~ 0
+RB14
+Text Label 1750 4200 0    50   ~ 0
+RD14
+Text Label 1750 4300 0    50   ~ 0
+RF4
+Text Label 2700 3600 0    50   ~ 0
+RA10
+Text Label 2700 3700 0    50   ~ 0
+RB9
+Text Label 2700 3800 0    50   ~ 0
+RB11
+Text Label 2700 3900 0    50   ~ 0
+RA1
+Text Label 2700 4000 0    50   ~ 0
+RF12
+Text Label 2700 4100 0    50   ~ 0
+RB13
+Text Label 2700 4200 0    50   ~ 0
+RB15
+Text Label 2700 4300 0    50   ~ 0
+RF5
+Text Label 4350 3300 0    50   ~ 0
+RE7
+Text Label 4350 3500 0    50   ~ 0
+RC2
+Text Label 4350 3700 0    50   ~ 0
+RC4
+Text Label 4350 3800 0    50   ~ 0
+RG7
+Text Label 4350 3900 0    50   ~ 0
+RA0
+Text Label 4350 4000 0    50   ~ 0
+RE9
+Text Label 4350 4100 0    50   ~ 0
+RB4
+Text Label 4350 4200 0    50   ~ 0
+RB2
+Text Label 4350 4300 0    50   ~ 0
+RB0
+Text Label 5250 3400 0    50   ~ 0
+RC1
+Text Label 5250 3600 0    50   ~ 0
+RC3
+Text Label 5250 3700 0    50   ~ 0
+RG6
+Text Label 5250 3800 0    50   ~ 0
+RG8
+Text Label 5250 3900 0    50   ~ 0
+RG9
+Text Label 5250 4000 0    50   ~ 0
+RE8
+Text Label 5250 4100 0    50   ~ 0
+RB5
+Text Label 5250 4200 0    50   ~ 0
+RB3
+Text Label 5250 4300 0    50   ~ 0
+RB1
+Text Label 4300 1550 0    50   ~ 0
+MCU_MISO
+Text Label 4300 1650 0    50   ~ 0
+LED1
+Text Label 4300 1850 0    50   ~ 0
+RA2
+Text Label 4350 2150 0    50   ~ 0
+RA4
+Text Label 4350 2250 0    50   ~ 0
+RA14
+Text Label 4350 2350 0    50   ~ 0
+RD10
+Text Label 4350 2450 0    50   ~ 0
+RD0
+Text Label 5250 1650 0    50   ~ 0
+LED2
+Text Label 5250 1850 0    50   ~ 0
+RF3
+Text Label 5250 1950 0    50   ~ 0
+MCU_SCK
+Text Label 5250 2050 0    50   ~ 0
+MCU_MOSI
+Text Label 5250 2150 0    50   ~ 0
+RA3
+Text Label 5250 2250 0    50   ~ 0
+RA5
+Text Label 5250 2350 0    50   ~ 0
+RA15
+Text Label 5250 2450 0    50   ~ 0
+RD9
+Text Label 1750 1250 0    50   ~ 0
+RD1
+Text Label 1750 1350 0    50   ~ 0
+RD3
+Text Label 1750 1450 0    50   ~ 0
+RD12
+Text Label 1750 1750 0    50   ~ 0
+RD4
+Text Label 1750 1850 0    50   ~ 0
+RF1
+Text Label 1750 2150 0    50   ~ 0
+RG12
+Text Label 1750 2250 0    50   ~ 0
+RE2
+Text Label 2700 1250 0    50   ~ 0
+RD2
+Text Label 2700 1350 0    50   ~ 0
+RD13
+Text Label 2700 1550 0    50   ~ 0
+RD5
+Text Label 2700 1850 0    50   ~ 0
+RD7
+Text Label 2700 1950 0    50   ~ 0
+RF0
+Text Label 2700 2050 0    50   ~ 0
+RE0
+Text Label 2700 2150 0    50   ~ 0
+RG14
+Text Label 2700 2450 0    50   ~ 0
+RE3
 $EndSCHEMATC
